File: hw/WiFi_module.brd (EAGLE design)
At the start: 25 x 45 mm, 22 parts, among them J1 GROVE-4P-2.0-3470130P1, J2 GROVE-4P-2.0-3470130P1

Commit message: Working on layout
Parts:
- added U$10: TI_CC3000, r2p_ic:TI_CC3000
- C1: value (none) -> 1u; device rcl:C1206 -> r2p_rcl:C1206
- C14, C17, C2, C3, C4, C6, C7, C8: device rcl:C0603 -> r2p_rcl:C0603
- C5: device rcl:C0805 -> r2p_rcl:C0805
- C9: value (none) -> 10u; device rcl:C0805 -> r2p_rcl:C0805
- J1, J2: value GROVE-4P-2.0-3470130P1 -> R2P_BUS-VERTICAL; device OPL Eagle Library:4P-2.0 -> r2p_connector:OPL-EAGLE-LIBRARY_4P-2.0
- LED1: device led:CHIPLED_0805 -> r2p_led:CHIPLED_0805
- R1: device rcl:R0603 -> r2p_rcl:R0603
- SOT1: device maxim:SOT23-8L -> r2p_ic:SOT23-8L
- U$2: device coilcraft:LPS4018 -> r2p_rcl:COILCRAFT_LPS4018
- U$3: device maxim:TDFN-10 -> r2p_ic:TDFN-10
- U$4: value FTSH-105TH -> JTAG-TH; device samtec:FTSH-105-TH -> r2p_connector:SAMTEC_FTSH-105-TH
- U$5: value ASD -> ABRACON_ASD; device abracon:2.5X2 -> r2p_ic:ABRACON_2.5X2
- U$6: value STM32F103CXTX -> STM32F303CTX; device st:LQFP48 -> r2p_ic:LQFP48
Connections:
- net VIN renamed +VBUS
- new net N$10: U$10.P$17
- new net N$13: U$10.P$19
- new net N$14: U$10.P$23
- new net N$15: U$10.P$24
- new net N$16: U$10.P$26
- new net N$17: U$10.P$27, U$10.P$28
- new net N$18: U$10.P$29, U$10.P$30
- new net N$21: U$10.P$35
- new net N$25: U$10.P$6
- new net N$26: U$10.P$8
- new net N$3: U$10.P$12
- new net N$5: U$10.P$13
- new net N$6: U$10.P$14
- new net N$9: U$10.P$15
- net GND: now also U$10.P$1, U$10.P$10, U$10.P$11, U$10.P$16, U$10.P$18, U$10.P$20, U$10.P$21, U$10.P$22, U$10.P$25, U$10.P$31, U$10.P$32, U$10.P$33, U$10.P$34, U$10.P$36, U$10.P$37, U$10.P$38, U$10.P$39, U$10.P$40, U$10.P$41, U$10.P$42, U$10.P$43, U$10.P$44, U$10.P$45, U$10.P$46, U$10.P$9

Commit message: Working on RF layout
Parts:
- added ANT1: ANT-2.4GHZ, r2p_rf:CHIP_ANTENNA_8X1
- added C10: 1uF, r2p_rcl:C0603
- added C11: 10uF, r2p_rcl:C0805
- added C12: 10pF, r2p_rcl:C0402
- added C13: 2.2pF, r2p_rcl:C0402
- added C15: DNP, r2p_rcl:C0402
- added L1: 2.2nH, r2p_rcl:L0402
- added L2: DNP, r2p_rcl:L0402
- added SJ1: (no value), SparkFun:SJ_3_PASTE1&2
- added U$11: U.FL, r2p_rf:U.FL
- added X1: MOLEX_53047-04, r2p_connector:MOLEX_53047-04
- U$10: value TI_CC3000 -> CC3000; device r2p_ic:TI_CC3000 -> r2p_rf:CC3000
- U$2: value LPS4018 -> (none)
Connections:
- removed net N$13: U$10.P$19
- removed net N$14: U$10.P$23
- removed net N$15: U$10.P$24
- removed net N$16: U$10.P$26
- removed net N$25: U$10.P$6
- removed net N$26: U$10.P$8
- new net DEBUG_RX: U$10.P$8, X1.4
- new net DEBUG_TX: U$10.P$6, X1.3
- new net SPI_CS: U$10.P$12, U$6.14
- new net SPI_IRQ: U$10.P$14, U$6.18
- new net SPI_MISO: U$10.P$13, U$6.16
- new net SPI_MOSI: U$10.P$15, U$6.17
- new net SPI_SCK: U$10.P$17, U$6.15
- new net SW_EN: U$10.P$26, U$6.12
- net +3V3: now also C10.1, C11.1, U$10.P$19, U$10.P$23
- net GND: now also C10.2, C11.2, L1.2, L2.2, SJ1.3, U$11.P$1, U$11.P$2, X1.2
- net N$10: now also C15.2, U$11.P$3; no longer U$10.P$17
- net N$21: now also C12.2
- net N$3: now also SJ1.1, U$10.P$7; no longer U$10.P$12
- net N$5: now also SJ1.2, U$10.P$5; no longer U$10.P$13
- net N$6: now also C12.1, C13.2, C15.1, L1.1; no longer U$10.P$14
- net N$9: now also ANT1.P$1, C13.1, L2.1; no longer U$10.P$15
Routing:
- net +3V3: track 78.8 -> 100.9 mm, vias 7 -> 8
- net SW_EN: track 0.00 -> 19.1 mm, vias 0 -> 2
- net SPI_CS: track 0.00 -> 10.4 mm, vias 0 -> 2
- net DEBUG_TX: track 0.00 -> 9.06 mm, vias 0 -> 1
- net DEBUG_RX: track 0.00 -> 8.17 mm
- net SPI_MISO: track 0.00 -> 7.55 mm, vias 0 -> 2
- net N$3: track 0.00 -> 5.27 mm
- net N$5: track 0.00 -> 4.69 mm
- net SPI_IRQ: track 0.00 -> 4.48 mm
- net SPI_MOSI: track 0.00 -> 3.95 mm
- net SPI_SCK: track 0.00 -> 2.73 mm
- net N$18: track 0.00 -> 1.20 mm
- net N$17: track 0.00 -> 1.20 mm

Commit message: Layout complete
Parts:
- moved C10 1.50 mm to (20.0, 24.2)
- moved C11 1.50 mm to (21.6, 24.2)
- moved C12 1.40 mm to (8.60, 40.5)
- moved U$10 1.40 mm to (11.6, 30.5)
- moved C15 1.15 mm to (6.85, 39.9)
- moved SJ1 1.12 mm to (2.30, 29.9), turned to 180 degrees
- moved U$11 1.12 mm to (2.80, 39.9)
- moved X1 0.28 mm to (2.30, 25.3)
- moved ANT1 0.20 mm to (19.5, 43.2)
- moved C13 0.20 mm to (12.4, 43.2)
- moved L1 0.20 mm to (10.6, 42.5)
- moved L2 0.20 mm to (14.2, 42.5)
Connections:
- net N$21: now also C15.1
- net N$6: no longer C15.1
Routing:
- net N$6: track 0.00 -> 2.79 mm
- net N$3: track 5.27 -> 3.61 mm
- net SPI_CS: track 10.4 -> 12.0 mm
- net SPI_MISO: track 7.55 -> 9.18 mm
- net DEBUG_RX: track 8.17 -> 6.76 mm
- net SPI_IRQ: track 4.48 -> 5.88 mm
- net SPI_MOSI: track 3.95 -> 5.18 mm
- net SPI_SCK: track 2.73 -> 3.72 mm
- net DEBUG_TX: track 9.06 -> 8.11 mm
- net +3V3: track 100.9 -> 100.1 mm
- added copper zone on layer 1, net N$10
- added copper zone on layer 1, net N$21
- added copper zone on layer 1, net N$6
- added copper zone on layer 1, net N$9

Commit message: Fixed silkscreen
Parts:
- U$5: value ABRACON_ASD -> OSC; device r2p_ic:ABRACON_2.5X2 -> r2p_ic:XTAL_2.5X2
Other:
- board text added: "RF module v1.0 (2015/02)"
- board text removed: "R2P module v0.0 (YYYY/MM)"
Changed lines of the file:
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@@
 <grid distance="0.5" unitdist="mm" unit="mm" style="dots" multiple="1" display="yes" altdistance="0.1" altunitdist="mm" altunit="mm"/>
 <layers>
-<layer number="1" name="Top" color="4" fill="1" visible="yes" active="yes"/>
-<layer number="16" name="Bottom" color="1" fill="1" visible="no" active="yes"/>
+<layer number="1" name="Top" color="4" fill="1" visible="no" active="yes"/>
+<layer number="16" name="Bottom" color="1" fill="1" visible="yes" active="yes"/>
 <layer number="17" name="Pads" color="2" fill="1" visible="yes" active="yes"/>
 <layer number="18" name="Vias" color="2" fill="1" visible="yes" active="yes"/>
 <layer number="19" name="Unrouted" color="6" fill="1" visible="yes" active="yes"/>
 <layer number="20" name="Dimension" color="15" fill="1" visible="yes" active="yes"/>
-<layer number="21" name="tPlace" color="7" fill="1" visible="yes" active="yes"/>
-<layer number="22" name="bPlace" color="7" fill="1" visible="no" active="yes"/>
-<layer number="23" name="tOrigins" color="15" fill="1" visible="yes" active="yes"/>
-<layer number="24" name="bOrigins" color="15" fill="1" visible="no" active="yes"/>
+<layer number="21" name="tPlace" color="7" fill="1" visible="no" active="yes"/>
+<layer number="22" name="bPlace" color="7" fill="1" visible="yes" active="yes"/>
+<layer number="23" name="tOrigins" color="15" fill="1" visible="no" active="yes"/>
+<layer number="24" name="bOrigins" color="15" fill="1" visible="yes" active="yes"/>
 <layer number="25" name="tNames" color="7" fill="1" visible="no" active="yes"/>
 <layer number="26" name="bNames" color="7" fill="1" visible="no" active="yes"/>
@@
 <layer number="37" name="tTest" color="7" fill="1" visible="no" active="yes"/>
 <layer number="38" name="bTest" color="7" fill="1" visible="no" active="yes"/>
-<layer number="39" name="tKeepout" color="4" fill="11" visible="yes" active="yes"/>
-<layer number="40" name="bKeepout" color="1" fill="11" visible="no" active="yes"/>
-<layer number="41" name="tRestrict" color="4" fill="10" visible="yes" active="yes"/>
-<layer number="42" name="bRestrict" color="1" fill="10" visible="no" active="yes"/>
+<layer number="39" name="tKeepout" color="4" fill="11" visible="no" active="yes"/>
+<layer number="40" name="bKeepout" color="1" fill="11" visible="yes" active="yes"/>
+<layer number="41" name="tRestrict" color="4" fill="10" visible="no" active="yes"/>
+<layer number="42" name="bRestrict" color="1" fill="10" visible="yes" active="yes"/>
 <layer number="43" name="vRestrict" color="2" fill="10" visible="no" active="yes"/>
 <layer number="44" name="Drills" color="7" fill="1" visible="no" active="yes"/>
@@
 <layer number="46" name="Milling" color="3" fill="1" visible="yes" active="yes"/>
 <layer number="47" name="Measures" color="7" fill="1" visible="yes" active="yes"/>
-<layer number="48" name="Document" color="7" fill="1" visible="yes" active="yes"/>
+<layer number="48" name="Document" color="7" fill="1" visible="no" active="yes"/>
 <layer number="49" name="Reference" color="7" fill="1" visible="no" active="yes"/>
 <layer number="50" name="dxf" color="7" fill="1" visible="no" active="no"/>
-<layer number="51" name="tDocu" color="7" fill="1" visible="yes" active="yes"/>
-<layer number="52" name="bDocu" color="7" fill="1" visible="no" active="yes"/>
+<layer number="51" name="tDocu" color="7" fill="1" visible="no" active="yes"/>
+<layer number="52" name="bDocu" color="7" fill="1" visible="yes" active="yes"/>
 <layer number="53" name="tGND_GNDA" color="7" fill="1" visible="no" active="no"/>
 <layer number="54" name="bGND_GNDA" color="7" fill="1" visible="no" active="no"/>
@@
 <layer number="155" name="FabDoc3" color="7" fill="1" visible="no" active="yes"/>
 <layer number="199" name="Contour" color="7" fill="1" visible="no" active="yes"/>
-<layer number="200" name="200bmp" color="7" fill="1" visible="no" active="yes"/>
+<layer number="200" name="200bmp" color="7" fill="1" visible="yes" active="yes"/>
 <layer number="201" name="201bmp" color="7" fill="1" visible="no" active="yes"/>
 <layer number="202" name="202bmp" color="7" fill="1" visible="no" active="yes"/>
@@
 <wire x1="6.55" y1="8" x2="6.55" y2="8.8" width="0.2" layer="41"/>
 <wire x1="6.55" y1="8.8" x2="7.45" y2="8.8" width="0.2" layer="41"/>
-<text x="4" y="6" size="1.5" layer="200" rot="MR90">R2P module
-v0.0 (YYYY/MM)</text>
+<text x="4" y="6" size="1.5" layer="200" rot="MR90">RF module
+v1.0 (2015/02)</text>
 <polygon width="0.2" layer="41">
 <vertex x="25" y="45"/>
@@
 </element>
 <element name="U$1" library="r2p_pcb" package="25X45" value="PCB_25X45" x="0" y="0" smashed="yes"/>
-<element name="U$5" library="r2p_ic" package="ABRACON_2.5X2" value="ABRACON_ASD" x="22.7" y="16" smashed="yes" rot="R180">
+<element name="U$5" library="r2p_ic" package="XTAL_2.5X2" value="OSC" x="22.7" y="16" smashed="yes" rot="R180">
 <attribute name="NAME" x="22.7" y="16" size="1" layer="25" font="vector" rot="R180" align="center"/>
 <attribute name="VALUE" x="24.95" y="18.75" size="1.27" layer="27" rot="R180"/>
