File: hw/WiFi_module.sch (EAGLE design)
At the start: 22 parts, among them J1 GROVE-4P-2.0-3470130P1, J2 GROVE-4P-2.0-3470130P1

Commit message: Working on layout
Parts:
- added U$10: TI_CC3000, r2p_ic:TI_CC3000
- C1: value (none) -> 1u; device rcl:C-EUC1206 -> r2p_rcl:C-1206
- C14, C17, C2, C3, C4, C6, C7, C8: device rcl:C-EUC0603 -> r2p_rcl:C-0603
- C5: device rcl:C-EUC0805 -> r2p_rcl:C-0805
- C9: value (none) -> 10u; device rcl:C-EUC0805 -> r2p_rcl:C-0805
- J1, J2: value GROVE-4P-2.0-3470130P1 -> R2P_BUS-VERTICAL; device OPL Eagle Library:GROVE-4P-2.0-3470130P1 -> r2p_connector:R2P_BUS-VERTICAL
- LED1: value (none) -> LED0805; device led:LEDCHIPLED_0805 -> r2p_led:LED0805
- R1: device rcl:R-EU_R0603 -> r2p_rcl:R-0603
- SOT1: device maxim:MAX3051EKA -> r2p_ic:MAX3051EKA
- U$2: device coilcraft:LPS4018 -> r2p_rcl:LPS4018
- U$3: device maxim:MAX17501 -> r2p_ic:MAX17501
- U$4: value FTSH-105TH -> JTAG-TH; device samtec:FTSH-105TH -> r2p_connector:JTAG-TH
- U$5: value ASD -> ABRACON_ASD; device abracon:ASD -> r2p_ic:ABRACON_ASD
- U$6: value STM32F103CXTX -> STM32F303CTX; device st:STM32F103CXTX -> r2p_ic:STM32F303CTX
Connections:
- net VIN renamed +VBUS
- new net N$10: U$10.SPI_CLK
- new net N$13: U$10.VBAT_IN
- new net N$14: U$10.VIO_HOST
- new net N$15: U$10.RESERVED_3
- new net N$16: U$10.VBAT_SW_EN
- new net N$17: U$10.SDA_CC3000, U$10.SDA_EEPROM
- new net N$18: U$10.SCL_CC3000, U$10.SCL_EEPROM
- new net N$21: U$10.RF_ANT
- new net N$25: U$10.WL_RS232_TX
- new net N$26: U$10.WL_RS232_RX
- new net N$3: U$10.SPI_CS
- new net N$5: U$10.SPI_DOUT
- new net N$6: U$10.SPI_IRQ
- new net N$9: U$10.SPI_DIN
- net +3V3: now also U$4.1; no longer U$4.P$1
- net GND: now also U$10.EXT_32K, U$10.GND@1, U$10.GND@10, U$10.GND@11, U$10.GND@12, U$10.GND@13, U$10.GND@14, U$10.GND@15, U$10.GND@16, U$10.GND@17, U$10.GND@18, U$10.GND@19, U$10.GND@2, U$10.GND@20, U$10.GND@21, U$10.GND@22, U$10.GND@23, U$10.GND@24, U$10.GND@3, U$10.GND@4, U$10.GND@5, U$10.GND@6, U$10.GND@7, U$10.GND@8, U$10.GND@9, U$4.3, U$4.5, U$4.7, U$4.9; no longer U$4.P$3, U$4.P$5, U$4.P$7, U$4.P$9
- net JTCK: now also U$4.4; no longer U$4.P$4
- net JTDI: now also U$4.8; no longer U$4.P$8
- net JTDO: now also U$4.6; no longer U$4.P$6
- net JTMS: now also U$4.2; no longer U$4.P$2
- net LED1: now also U$6.PF1/OSC_OUT; no longer U$6.PD1/OSC_OUT
- net NRST: now also U$4.10; no longer U$4.P$10
- net OSC_IN: now also U$6.PF0/OSC_IN; no longer U$6.PD0/OSC_IN

Commit message: Working on RF layout
Parts:
- added ANT1: ANT-2.4GHZ, r2p_rf:ANT-2.4GHZ
- added C10: 1uF, r2p_rcl:C0603
- added C11: 10uF, r2p_rcl:C0805
- added C12: 10pF, r2p_rcl:C0402
- added C13: 2.2pF, r2p_rcl:C0402
- added C15: DNP, r2p_rcl:C0402
- added L1: 2.2nH, r2p_rcl:L0402
- added L2: DNP, r2p_rcl:L0402
- added SJ1: (no value), SparkFun:SOLDERJUMPER_2WAYPASTE1&2
- added U$11: U.FL, r2p_rf:U.FL
- added X1: MOLEX_53047-04, r2p_connector:MOLEX_53047-04
- C1: device r2p_rcl:C-1206 -> r2p_rcl:C1206
- C14, C17, C2, C3, C4, C6, C7, C8: device r2p_rcl:C-0603 -> r2p_rcl:C0603
- C5, C9: device r2p_rcl:C-0805 -> r2p_rcl:C0805
- R1: device r2p_rcl:R-0603 -> r2p_rcl:R0603
- U$10: value TI_CC3000 -> CC3000; device r2p_ic:TI_CC3000 -> r2p_rf:CC3000
- U$2: value LPS4018 -> (none)
Connections:
- removed net N$13: U$10.VBAT_IN
- removed net N$14: U$10.VIO_HOST
- removed net N$15: U$10.RESERVED_3
- removed net N$16: U$10.VBAT_SW_EN
- removed net N$25: U$10.WL_RS232_TX
- removed net N$26: U$10.WL_RS232_RX
- new net DEBUG_RX: U$10.WL_RS232_RX, X14.S
- new net DEBUG_TX: U$10.WL_RS232_TX, X13.S
- new net SPI_CS: U$10.SPI_CS, U$6.PA4
- new net SPI_IRQ: U$10.SPI_IRQ, U$6.PB0
- new net SPI_MISO: U$10.SPI_DOUT, U$6.PA6
- new net SPI_MOSI: U$10.SPI_DIN, U$6.PA7
- new net SPI_SCK: U$10.SPI_CLK, U$6.PA5
- new net SW_EN: U$10.VBAT_SW_EN, U$6.PA2
- net +3V3: now also C10.1, C11.1, U$10.VBAT_IN, U$10.VIO_HOST
- net GND: now also C10.2, C11.2, L1.2, L2.2, SJ1.3, U$11.GND@0, U$11.GND@1, X12.S
- net N$10: now also C15.2, U$11.SIGNAL; no longer U$10.SPI_CLK
- net N$21: now also C12.2
- net N$3: now also SJ1.1, U$10.WL_EN1; no longer U$10.SPI_CS
- net N$5: now also SJ1.2, U$10.WL_EN2; no longer U$10.SPI_DOUT
- net N$6: now also C12.1, C13.2, C15.1, L1.1; no longer U$10.SPI_IRQ
- net N$9: now also ANT1.P$1, C13.1, L2.1; no longer U$10.SPI_DIN

Commit message: Layout complete
Connections:
- net N$21: now also C15.1
- net N$6: no longer C15.1
Other:
- moved on the sheet: ANT1, C12, C13, L1, L2
Changed lines of the file:
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@@
 <instance part="X1" gate="4" x="185.42" y="111.76"/>
 <instance part="GND25" gate="1" x="180.34" y="106.68"/>
-<instance part="GND26" gate="1" x="218.44" y="193.04"/>
-<instance part="GND27" gate="1" x="205.74" y="193.04"/>
-<instance part="C12" gate="G$1" x="231.14" y="205.74"/>
-<instance part="C13" gate="G$1" x="210.82" y="210.82" rot="R90"/>
-<instance part="L1" gate="G$1" x="218.44" y="203.2"/>
-<instance part="L2" gate="G$1" x="205.74" y="203.2"/>
-<instance part="ANT1" gate="G$1" x="205.74" y="220.98"/>
+<instance part="GND26" gate="1" x="218.44" y="205.74"/>
+<instance part="GND27" gate="1" x="205.74" y="205.74"/>
+<instance part="C12" gate="G$1" x="231.14" y="218.44"/>
+<instance part="C13" gate="G$1" x="210.82" y="223.52" rot="R90"/>
+<instance part="L1" gate="G$1" x="218.44" y="215.9"/>
+<instance part="L2" gate="G$1" x="205.74" y="215.9"/>
+<instance part="ANT1" gate="G$1" x="205.74" y="233.68"/>
 <instance part="U$11" gate="G$1" x="251.46" y="210.82" rot="MR0"/>
 <instance part="C15" gate="G$1" x="238.76" y="210.82" rot="R90"/>
@@
 <segment>
 <pinref part="U$10" gate="G$1" pin="RF_ANT"/>
-<wire x1="231.14" y1="190.5" x2="231.14" y2="200.66" width="0.1524" layer="91"/>
+<wire x1="231.14" y1="190.5" x2="231.14" y2="210.82" width="0.1524" layer="91"/>
 <pinref part="C12" gate="G$1" pin="2"/>
+<pinref part="C15" gate="G$1" pin="1"/>
+<wire x1="231.14" y1="210.82" x2="231.14" y2="213.36" width="0.1524" layer="91"/>
+<wire x1="236.22" y1="210.82" x2="231.14" y2="210.82" width="0.1524" layer="91"/>
+<junction x="231.14" y="210.82"/>
 </segment>
 </net>
@@
 <net name="N$6" class="0">
 <segment>
-<wire x1="215.9" y1="210.82" x2="218.44" y2="210.82" width="0.1524" layer="91"/>
-<wire x1="218.44" y1="210.82" x2="231.14" y2="210.82" width="0.1524" layer="91"/>
-<wire x1="231.14" y1="210.82" x2="231.14" y2="208.28" width="0.1524" layer="91"/>
+<wire x1="215.9" y1="223.52" x2="218.44" y2="223.52" width="0.1524" layer="91"/>
+<wire x1="218.44" y1="223.52" x2="231.14" y2="223.52" width="0.1524" layer="91"/>
+<wire x1="231.14" y1="223.52" x2="231.14" y2="220.98" width="0.1524" layer="91"/>
 <pinref part="C12" gate="G$1" pin="1"/>
 <pinref part="C13" gate="G$1" pin="2"/>
 <pinref part="L1" gate="G$1" pin="1"/>
-<junction x="218.44" y="210.82"/>
-<pinref part="C15" gate="G$1" pin="1"/>
-<wire x1="236.22" y1="210.82" x2="231.14" y2="210.82" width="0.1524" layer="91"/>
-<junction x="231.14" y="210.82"/>
+<junction x="218.44" y="223.52"/>
 </segment>
 </net>
 <net name="N$9" class="0">
 <segment>
-<wire x1="208.28" y1="210.82" x2="205.74" y2="210.82" width="0.1524" layer="91"/>
+<wire x1="208.28" y1="223.52" x2="205.74" y2="223.52" width="0.1524" layer="91"/>
 <pinref part="C13" gate="G$1" pin="1"/>
 <pinref part="L2" gate="G$1" pin="1"/>
-<wire x1="205.74" y1="210.82" x2="205.74" y2="215.9" width="0.1524" layer="91"/>
-<junction x="205.74" y="210.82"/>
+<wire x1="205.74" y1="223.52" x2="205.74" y2="228.6" width="0.1524" layer="91"/>
+<junction x="205.74" y="223.52"/>
 <pinref part="ANT1" gate="G$1" pin="P$1"/>
 </segment>

Commit message: Fixed silkscreen
Parts:
- U$5: value ABRACON_ASD -> OSC; device r2p_ic:ABRACON_ASD -> r2p_ic:OSC
Changed lines of the file:
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@@
 <part name="SOT1" library="r2p_ic" deviceset="MAX3051" device="EKA"/>
 <part name="U$1" library="r2p_pcb" deviceset="PCB_25X45" device=""/>
-<part name="U$5" library="r2p_ic" deviceset="ABRACON_ASD" device=""/>
+<part name="U$5" library="r2p_ic" deviceset="OSC" device=""/>
 <part name="+3V7" library="r2p_supply" deviceset="+3V3" device=""/>
 <part name="U$7" library="r2p_supply" deviceset="+VBUS" device=""/>
